Commit message: Fix G1 bringup and setup issues

File: description_files/urdf/g1_29dof.urdf (robot description, URDF)
Before this commit: robot g1_29dof_rev_1_0, 57 links, 56 joints
Joints:
- joint livox_joint: origin xyz=0.0 0.0 0.0 rpy=3.141561 0 0 -> xyz=0.0 0.0 0.0 rpy=0 0 0
- joint mid360_joint: origin xyz=0.0002835 0.00003 0.41618 rpy=0 0.04014257279586953 0 -> xyz=0.0002835 0.00003 0.428434 rpy=3.141592653589793 0.05112069379091391 0

File: description_files/urdf/g1_29dof_dx3.urdf (robot description, URDF)
Before this commit: robot g1_29dof_with_hand_rev_1_0, 53 links, 52 joints
Links:
- added link left_hand_point_contact
- added link livox_frame
- added link right_hand_point_contact
Joints:
- added joint left_hand_point_contact_fix_joint: type fixed, parent left_hand_palm_link, child left_hand_point_contact, origin xyz=0.05 0.0 0.0 rpy=0 0 0
- added joint livox_joint: type fixed, parent mid360_link, child livox_frame, origin xyz=0.0 0.0 0.0 rpy=0 0 0
- added joint right_hand_point_contact_fix_joint: type fixed, parent right_hand_palm_link, child right_hand_point_contact, origin xyz=0.05 0.0 0.0 rpy=0 0 0
- joint mid360_joint: origin xyz=0.0002835 0.00003 0.41618 rpy=0 0.04014257279586953 0 -> xyz=0.0002835 0.00003 0.428434 rpy=3.141592653589793 0.05112069379091391 0

File: description_files/urdf/g1_29dof_dx3_upperbody.urdf (robot description, URDF)
Before this commit: robot g1_29dof_with_hand_rev_1_0, 40 links, 39 joints
Links:
- added link left_hand_point_contact
- added link livox_frame
- added link right_hand_point_contact
- link head_link: geometry collision mesh filename=package://g1pilot/description_files/meshes/head_link.STL; visual mesh filename=package://g1pilot/description_files/meshes/head_link.STL
- link left_elbow_link: geometry collision mesh filename=package://g1pilot/description_files/meshes/left_elbow_link.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; visual mesh filename=package://g1pilot/description_files/meshes/left_elbow_link.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
- link left_hand_index_0_link: geometry collision mesh filename=package://g1pilot/description_files/meshes/left_hand_index_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; visual mesh filename=package://g1pilot/description_files/meshes/left_hand_index_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
- link left_hand_index_1_link: geometry collision mesh filename=package://g1pilot/description_files/meshes/left_hand_index_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; visual mesh filename=package://g1pilot/description_files/meshes/left_hand_index_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
- link left_hand_middle_0_link: geometry collision mesh filename=package://g1pilot/description_files/meshes/left_hand_middle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; visual mesh filename=package://g1pilot/description_files/meshes/left_hand_middle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
- link left_hand_middle_1_link: geometry collision mesh filename=package://g1pilot/description_files/meshes/left_hand_middle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; visual mesh filename=package://g1pilot/description_files/meshes/left_hand_middle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
- link left_hand_palm_link: geometry collision mesh filename=package://g1pilot/description_files/meshes/left_hand_palm_l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; visual mesh filename=package://g1pilot/description_files/meshes/left_hand_palm_l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
- link left_hand_thumb_0_link: geometry collision mesh filename=package://g1pilot/description_files/meshes/left_hand_thumb_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; visual mesh filename=package://g1pilot/description_files/meshes/left_hand_thumb_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
- link left_hand_thumb_1_link: geometry collision box size=0.02 0.03 0.02; visual mesh filename=package://g1pilot/description_files/meshes/left_hand_thumb_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
- link left_hand_thumb_2_link: geometry collision mesh filename=package://g1pilot/description_files/meshes/left_hand_thumb_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; visual mesh filename=package://g1pilot/description_files/meshes/left_hand_thumb_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
- link left_shoulder_pitch_link: geometry collision cylinder length=0.05 radius=0.03; visual mesh filename=package://g1pilot/description_files/meshes/left_shoulder_pi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
- link left_shoulder_roll_link: geometry collision cylinder length=0.03 radius=0.03; visual mesh filename=package://g1pilot/description_files/meshes/left_shoulder_ro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
- link left_shoulder_yaw_link: geometry collision mesh filename=package://g1pilot/description_files/meshes/left_shoulder_ya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; visual mesh filename=package://g1pilot/description_files/meshes/left_shoulder_ya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
- link left_wrist_pitch_link: geometry collision mesh filename=package://g1pilot/description_files/meshes/left_wrist_pitch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; visual mesh filename=package://g1pilot/description_files/meshes/left_wrist_pitch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
- link left_wrist_roll_link: geometry collision mesh filename=package://g1pilot/description_files/meshes/left_wrist_roll_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; visual mesh filename=package://g1pilot/description_files/meshes/left_wrist_roll_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
- link left_wrist_yaw_link: geometry collision mesh filename=package://g1pilot/description_files/meshes/left_wrist_yaw_l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; visual mesh filename=package://g1pilot/description_files/meshes/left_wrist_yaw_l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
- link logo_link: geometry collision mesh filename=package://g1pilot/description_files/meshes/logo_link.STL; visual mesh filename=package://g1pilot/description_files/meshes/logo_link.STL
- link pelvis: geometry visual mesh filename=package://g1pilot/description_files/meshes/pelvis.STL
- link right_elbow_link: geometry collision mesh filename=package://g1pilot/description_files/meshes/right_elbow_link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; visual mesh filename=package://g1pilot/description_files/meshes/right_elbow_link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
- link right_hand_index_0_link: geometry collision mesh filename=package://g1pilot/description_files/meshes/right_hand_index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; visual mesh filename=package://g1pilot/description_files/meshes/right_hand_index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
- link right_hand_index_1_link: geometry collision mesh filename=package://g1pilot/description_files/meshes/right_hand_index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; visual mesh filename=package://g1pilot/description_files/meshes/right_hand_index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
- link right_hand_middle_0_link: geometry collision mesh filename=package://g1pilot/description_files/meshes/right_hand_middl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; visual mesh filename=package://g1pilot/description_files/meshes/right_hand_middl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
- link right_hand_middle_1_link: geometry collision mesh filename=package://g1pilot/description_files/meshes/right_hand_middl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; visual mesh filename=package://g1pilot/description_files/meshes/right_hand_middl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
- link right_hand_palm_link: geometry collision mesh filename=package://g1pilot/description_files/meshes/right_hand_palm_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; visual mesh filename=package://g1pilot/description_files/meshes/right_hand_palm_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
- link right_hand_thumb_0_link: geometry collision mesh filename=package://g1pilot/description_files/meshes/right_hand_thumb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; visual mesh filename=package://g1pilot/description_files/meshes/right_hand_thumb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
- link right_hand_thumb_1_link: geometry collision box size=0.02 0.03 0.02; visual mesh filename=package://g1pilot/description_files/meshes/right_hand_thumb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
- link right_hand_thumb_2_link: geometry collision mesh filename=package://g1pilot/description_files/meshes/right_hand_thumb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; visual mesh filename=package://g1pilot/description_files/meshes/right_hand_thumb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
- link right_shoulder_pitch_link: geometry collision cylinder length=0.05 radius=0.03; visual mesh filename=package://g1pilot/description_files/meshes/right_shoulder_p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
- link right_shoulder_roll_link: geometry collision cylinder length=0.03 radius=0.03; visual mesh filename=package://g1pilot/description_files/meshes/right_shoulder_r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
- link right_shoulder_yaw_link: geometry collision mesh filename=package://g1pilot/description_files/meshes/right_shoulder_y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; visual mesh filename=package://g1pilot/description_files/meshes/right_shoulder_y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
- link right_wrist_pitch_link: geometry collision mesh filename=package://g1pilot/description_files/meshes/right_wrist_pitc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; visual mesh filename=package://g1pilot/description_files/meshes/right_wrist_pitc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
- link right_wrist_roll_link: geometry collision mesh filename=package://g1pilot/description_files/meshes/right_wrist_roll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; visual mesh filename=package://g1pilot/description_files/meshes/right_wrist_roll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
- link right_wrist_yaw_link: geometry collision mesh filename=package://g1pilot/description_files/meshes/right_wrist_yaw_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; visual mesh filename=package://g1pilot/description_files/meshes/right_wrist_yaw_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
- link torso_link: geometry collision mesh filename=package://g1pilot/description_files/meshes/torso_link_rev_1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; visual mesh filename=package://g1pilot/description_files/meshes/torso_link_rev_1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
- link waist_roll_link: geometry visual mesh filename=package://g1pilot/description_files/meshes/waist_roll_link_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
- link waist_yaw_link: geometry visual mesh filename=package://g1pilot/description_files/meshes/waist_yaw_link_r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
Joints:
- added joint left_hand_point_contact_fix_joint: type fixed, parent left_hand_palm_link, child left_hand_point_contact, origin xyz=0.05 0.0 0.0 rpy=0 0 0
- added joint livox_joint: type fixed, parent mid360_link, child livox_frame, origin xyz=0.0 0.0 0.0 rpy=0 0 0
- added joint right_hand_point_contact_fix_joint: type fixed, parent right_hand_palm_link, child right_hand_point_contact, origin xyz=0.05 0.0 0.0 rpy=0 0 0
- joint mid360_joint: origin xyz=0.0002835 0.00003 0.41618 rpy=0 0.04014257279586953 0 -> xyz=0.0002835 0.00003 0.428434 rpy=3.141592653589793 0.05112069379091391 0

File: description_files/urdf/g1_29dof_upperbody.urdf (robot description, URDF)
Before this commit: robot g1_29dof_rev_1_0, 30 links, 29 joints
Joints:
- joint livox_joint: origin xyz=0.0 0.0 0.0 rpy=3.141561 0 0 -> xyz=0.0 0.0 0.0 rpy=0 0 0
- joint mid360_joint: origin xyz=0.0002835 0.00003 0.41618 rpy=0 0.04014257279586953 0 -> xyz=0.0002835 0.00003 0.428434 rpy=3.141592653589793 0.05112069379091391 0
