Commit message: Add G1Pilot lab integration and MuJoCo Dex3 backend
Integrate SDK arm and hand commands with a locked-waist MuJoCo plant and OpenHomie leg policy. Include simulation launch wiring, model generation, reachability support and native ROS setup fixes.

Consolidate the fork's six development commits on the upstream base. Retain public setup instructions and upstream attribution; exclude private running notes from the new development history.

File: description_files/urdf/g1_29dof_lock_waist.urdf (robot description, URDF)
Before this commit: robot g1_29dof_with_hand_rev_1_0, 43 links, 42 joints
Links:
- removed link left_hand_index_0_link
- removed link left_hand_index_1_link
- removed link left_hand_middle_0_link
- removed link left_hand_middle_1_link
- removed link left_hand_palm_link
- removed link left_hand_thumb_0_link
- removed link left_hand_thumb_1_link
- removed link left_hand_thumb_2_link
- removed link right_hand_index_0_link
- removed link right_hand_index_1_link
- removed link right_hand_middle_0_link
- removed link right_hand_middle_1_link
- removed link right_hand_palm_link
- removed link right_hand_thumb_0_link
- removed link right_hand_thumb_1_link
- removed link right_hand_thumb_2_link
- added link left_ankle_pitch_link, mass 0.074; collision mesh filename=package://g1pilot/description_files/meshes/left_ankle_pitch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; visual mesh filename=package://g1pilot/description_files/meshes/left_ankle_pitch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
- added link left_ankle_roll_link, mass 0.608; collision sphere radius=0.005; collision sphere radius=0.005
- added link left_hip_pitch_link, mass 1.35; collision cylinder length=0.08 radius=0.04; visual mesh filename=package://g1pilot/description_files/meshes/left_hip_pitch_l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
- added link left_hip_roll_link, mass 1.52; collision cylinder length=0.12 radius=0.07; visual mesh filename=package://g1pilot/description_files/meshes/left_hip_roll_li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
- added link left_hip_yaw_link, mass 1.702; collision cylinder length=0.18 radius=0.055; visual mesh filename=package://g1pilot/description_files/meshes/left_hip_yaw_lin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
- added link left_knee_link, mass 1.932; collision cylinder length=0.30 radius=0.06; visual mesh filename=package://g1pilot/description_files/meshes/left_knee_link.S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
- added link left_rubber_hand, mass 0.170; collision box size=0.15 0.08 0.12; visual mesh filename=package://g1pilot/description_files/meshes/left_rubber_hand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
- added link pelvis_contour_link, mass 0.001; collision box size=0.12 0.14 0.12; visual mesh filename=package://g1pilot/description_files/meshes/pelvis_contour_l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
- added link right_ankle_pitch_link, mass 0.074; collision mesh filename=package://g1pilot/description_files/meshes/right_ankle_pitc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; visual mesh filename=package://g1pilot/description_files/meshes/right_ankle_pitc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
- added link right_ankle_roll_link, mass 0.608; collision sphere radius=0.005; collision sphere radius=0.005
- added link right_hip_pitch_link, mass 1.35; collision cylinder length=0.08 radius=0.04; visual mesh filename=package://g1pilot/description_files/meshes/right_hip_pitch_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
- added link right_hip_roll_link, mass 1.52; collision cylinder length=0.12 radius=0.07; visual mesh filename=package://g1pilot/description_files/meshes/right_hip_roll_l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
- added link right_hip_yaw_link, mass 1.702; collision cylinder length=0.18 radius=0.055; visual mesh filename=package://g1pilot/description_files/meshes/right_hip_yaw_li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
- added link right_knee_link, mass 1.932; collision cylinder length=0.30 radius=0.06; visual mesh filename=package://g1pilot/description_files/meshes/right_knee_link.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
- added link right_rubber_hand, mass 0.170; collision box size=0.15 0.08 0.12; visual mesh filename=package://g1pilot/description_files/meshes/right_rubber_han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
- added link world
- link left_elbow_link: geometry collision cylinder length=0.13 radius=0.035; visual mesh filename=package://g1pilot/description_files/meshes/left_elbow_link.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
- link left_shoulder_yaw_link: geometry collision cylinder length=0.145 radius=0.04; visual mesh filename=package://g1pilot/description_files/meshes/left_shoulder_ya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
- link left_wrist_pitch_link: geometry collision cylinder length=0.10 radius=0.03; visual mesh filename=package://g1pilot/description_files/meshes/left_wrist_pitch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
- link left_wrist_roll_link: geometry collision cylinder length=0.056 radius=0.03; visual mesh filename=package://g1pilot/description_files/meshes/left_wrist_roll_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
- link left_wrist_yaw_link: geometry collision cylinder length=0.06 radius=0.03; visual mesh filename=package://g1pilot/description_files/meshes/left_wrist_yaw_l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
- link right_elbow_link: geometry collision cylinder length=0.13 radius=0.035; visual mesh filename=package://g1pilot/description_files/meshes/right_elbow_link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
- link right_shoulder_yaw_link: geometry collision cylinder length=0.145 radius=0.04; visual mesh filename=package://g1pilot/description_files/meshes/right_shoulder_y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
- link right_wrist_pitch_link: geometry collision cylinder length=0.10 radius=0.03; visual mesh filename=package://g1pilot/description_files/meshes/right_wrist_pitc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
- link right_wrist_roll_link: geometry collision cylinder length=0.056 radius=0.03; visual mesh filename=package://g1pilot/description_files/meshes/right_wrist_roll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
- link right_wrist_yaw_link: geometry collision cylinder length=0.06 radius=0.03; visual mesh filename=package://g1pilot/description_files/meshes/right_wrist_yaw_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
- link torso_link: geometry collision box size=0.13 0.20 0.30; visual mesh filename=package://g1pilot/description_files/meshes/torso_link_rev_1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
- link waist_roll_link: geometry collision cylinder length=0.024 radius=0.017; visual mesh filename=package://g1pilot/description_files/meshes/waist_roll_link_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
- link waist_yaw_link: geometry collision cylinder length=0.15 radius=0.06; visual mesh filename=package://g1pilot/description_files/meshes/waist_yaw_link_r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
Joints:
- removed joint left_hand_index_0_joint
- removed joint left_hand_index_1_joint
- removed joint left_hand_middle_0_joint
- removed joint left_hand_middle_1_joint
- removed joint left_hand_thumb_0_joint
- removed joint left_hand_thumb_1_joint
- removed joint left_hand_thumb_2_joint
- removed joint right_hand_index_0_joint
- removed joint right_hand_index_1_joint
- removed joint right_hand_middle_0_joint
- removed joint right_hand_middle_1_joint
- removed joint right_hand_thumb_0_joint
- removed joint right_hand_thumb_1_joint
- removed joint right_hand_thumb_2_joint
- added joint floating_base_joint: type floating, parent world, child pelvis
- added joint left_ankle_pitch_joint: type revolute, parent left_knee_link, child left_ankle_pitch_link, origin xyz=0 -9.4445E-05 -0.30001 rpy=0 0 0, axis 0 1 0, limit lower=-0.87267 upper=0.5236 effort=35 velocity=30
- added joint left_ankle_roll_joint: type revolute, parent left_ankle_pitch_link, child left_ankle_roll_link, origin xyz=0 0 -0.017558 rpy=0 0 0, axis 1 0 0, limit lower=-0.2618 upper=0.2618 effort=35 velocity=30
- added joint left_hip_pitch_joint: type revolute, parent pelvis, child left_hip_pitch_link, origin xyz=0 0.064452 -0.1027 rpy=0 0 0, axis 0 1 0, limit lower=-2.5307 upper=2.8798 effort=88 velocity=32
- added joint left_hip_roll_joint: type revolute, parent left_hip_pitch_link, child left_hip_roll_link, origin xyz=0 0.052 -0.030465 rpy=0 -0.1749 0, axis 1 0 0, limit lower=-0.5236 upper=2.9671 effort=139 velocity=20
- added joint left_hip_yaw_joint: type revolute, parent left_hip_roll_link, child left_hip_yaw_link, origin xyz=0.025001 0 -0.12412 rpy=0 0 0, axis 0 0 1, limit lower=-2.7576 upper=2.7576 effort=88 velocity=32
- added joint left_knee_joint: type revolute, parent left_hip_yaw_link, child left_knee_link, origin xyz=-0.078273 0.0021489 -0.17734 rpy=0 0.1749 0, axis 0 1 0, limit lower=-0.087267 upper=2.8798 effort=139 velocity=20
- added joint pelvis_contour_joint: type fixed, parent pelvis, child pelvis_contour_link
- added joint right_ankle_pitch_joint: type revolute, parent right_knee_link, child right_ankle_pitch_link, origin xyz=0 9.4445E-05 -0.30001 rpy=0 0 0, axis 0 1 0, limit lower=-0.87267 upper=0.5236 effort=35 velocity=30
- added joint right_ankle_roll_joint: type revolute, parent right_ankle_pitch_link, child right_ankle_roll_link, origin xyz=0 0 -0.017558 rpy=0 0 0, axis 1 0 0, limit lower=-0.2618 upper=0.2618 effort=35 velocity=30
- added joint right_hip_pitch_joint: type revolute, parent pelvis, child right_hip_pitch_link, origin xyz=0 -0.064452 -0.1027 rpy=0 0 0, axis 0 1 0, limit lower=-2.5307 upper=2.8798 effort=88 velocity=32
- added joint right_hip_roll_joint: type revolute, parent right_hip_pitch_link, child right_hip_roll_link, origin xyz=0 -0.052 -0.030465 rpy=0 -0.1749 0, axis 1 0 0, limit lower=-2.9671 upper=0.5236 effort=139 velocity=20
- added joint right_hip_yaw_joint: type revolute, parent right_hip_roll_link, child right_hip_yaw_link, origin xyz=0.025001 0 -0.12412 rpy=0 0 0, axis 0 0 1, limit lower=-2.7576 upper=2.7576 effort=88 velocity=32
- added joint right_knee_joint: type revolute, parent right_hip_yaw_link, child right_knee_link, origin xyz=-0.078273 -0.0021489 -0.17734 rpy=0 0.1749 0, axis 0 1 0, limit lower=-0.087267 upper=2.8798 effort=139 velocity=20
- joint left_hand_palm_joint: child left_hand_palm_link -> left_rubber_hand
- joint left_hand_point_contact_fix_joint: parent left_hand_palm_link -> left_rubber_hand
- joint right_hand_palm_joint: child right_hand_palm_link -> right_rubber_hand
- joint right_hand_point_contact_fix_joint: parent right_hand_palm_link -> right_rubber_hand
- joint waist_pitch_joint: type revolute -> fixed
- joint waist_roll_joint: type revolute -> fixed
